File: demo1.kicad_sch (KiCad schematic)
At the start: 15 parts, among them J1 Screw_Terminal_01x12, J2 Screw_Terminal_01x12, K1 SANYOU_SRD_Form_A, K2 SANYOU_SRD_Form_A, K3 SANYOU_SRD_Form_A, K4 SANYOU_SRD_Form_A, SW1 SW_EMER_BACK, SW2 SW_EMER_DRIVER, SW3 SW_EMER_DRIVER2

Commit message: Update demo1.kicad_sch
Other:
- note removed: "32"
- note removed: "34"
- note removed: "ECU"
- note removed: "IG#1/2 IN"

Commit message: Update demo1.kicad_sch (latest)
Parts:
- added L2: L, symbol Device:L
Connections:
- net GND: now also L2.2
- net at K1.3: now also L1.1, L2.1
Other:
- note added: "32"
- note added: "ignition coil-1"
- note added: "ignition coil-2"
- note removed: "33"
Changed lines of the file:
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@@
 		)
 	)
-	(text "33\n"
-		(exclude_from_sim no)
-		(at 216.916 92.202 0)
+	(text "32"
+		(exclude_from_sim no)
+		(at 208.28 92.202 0)
 		(effects
 			(font
@@
 		)
 	)
+	(text "ignition\ncoil-1\n"
+		(exclude_from_sim no)
+		(at 211.836 103.124 0)
+		(effects
+			(font
+				(size 1.27 1.27)
+			)
+		)
+	)
 	(text "16"
 		(exclude_from_sim no)
@@
 		(exclude_from_sim no)
 		(at 201.676 81.534 0)
+		(effects
+			(font
+				(size 1.27 1.27)
+			)
+		)
+	)
+	(text "ignition\ncoil-2\n"
+		(exclude_from_sim no)
+		(at 221.742 103.378 0)
 		(effects
 			(font
@@
 	)
 	(junction
+		(at 190.5 40.64)
+		(diameter 0)
+		(color 0 0 0 0)
+	)
+	(junction
 		(at 123.19 87.63)
 		(diameter 0)
@@
 	)
 	(junction
-		(at 205.74 95.25)
-		(diameter 0)
-		(color 0 0 0 0)
-	)
-	(junction
 		(at 250.19 96.52)
 		(diameter 0)
@@
 	)
 	(junction
+		(at 205.74 97.79)
+		(diameter 0)
+		(color 0 0 0 0)
+	)
+	(junction
+		(at 201.93 105.41)
+		(diameter 0)
+		(color 0 0 0 0)
+	)
+	(junction
 		(at 114.3 64.77)
 		(diameter 0)
@@
 	)
 	(junction
+		(at 205.74 105.41)
+		(diameter 0)
+		(color 0 0 0 0)
+	)
+	(junction
 		(at 270.51 74.93)
 		(diameter 0)
@@
 	)
 	(junction
+		(at 205.74 93.98)
+		(diameter 0)
+		(color 0 0 0 0)
+	)
+	(junction
 		(at 270.51 69.85)
 		(diameter 0)
@@
 	(wire
 		(pts
+			(xy 205.74 105.41) (xy 215.9 105.41)
+		)
+		(stroke
+			(width 0)
+			(type default)
+		)
+	)
+	(wire
+		(pts
 			(xy 105.41 113.03) (xy 102.87 113.03)
 		)
@@
 	(wire
 		(pts
-			(xy 102.87 40.64) (xy 194.31 40.64)
+			(xy 102.87 40.64) (xy 190.5 40.64)
 		)
 		(stroke
@@
 	(wire
 		(pts
-			(xy 205.74 95.25) (xy 205.74 97.79)
-		)
-		(stroke
-			(width 0)
-			(type default)
-		)
-	)
-	(wire
-		(pts
 			(xy 76.2 123.19) (xy 85.09 123.19)
 		)
@@
 	(wire
 		(pts
+			(xy 201.93 109.22) (xy 201.93 105.41)
+		)
+		(stroke
+			(width 0)
+			(type default)
+		)
+	)
+	(wire
+		(pts
 			(xy 228.6 82.55) (xy 242.57 82.55)
 		)
@@
 	(wire
 		(pts
-			(xy 205.74 105.41) (xy 190.5 105.41)
+			(xy 205.74 105.41) (xy 201.93 105.41)
+		)
+		(stroke
+			(width 0)
+			(type default)
+		)
+	)
+	(wire
+		(pts
+			(xy 210.82 90.17) (xy 210.82 93.98)
 		)
 		(stroke
@@
 	(wire
 		(pts
+			(xy 205.74 97.79) (xy 215.9 97.79)
+		)
+		(stroke
+			(width 0)
+			(type default)
+		)
+	)
+	(wire
+		(pts
 			(xy 264.16 90.17) (xy 270.51 90.17)
 		)
@@
 	(wire
 		(pts
-			(xy 218.44 90.17) (xy 218.44 95.25)
-		)
-		(stroke
-			(width 0)
-			(type default)
-		)
-	)
-	(wire
-		(pts
 			(xy 237.49 88.9) (xy 237.49 123.19)
 		)
@@
 	(wire
 		(pts
+			(xy 190.5 93.98) (xy 205.74 93.98)
+		)
+		(stroke
+			(width 0)
+			(type default)
+		)
+	)
+	(wire
+		(pts
 			(xy 248.92 90.17) (xy 248.92 107.95)
 		)
@@
 	(wire
 		(pts
+			(xy 227.33 109.22) (xy 201.93 109.22)
+		)
+		(stroke
+			(width 0)
+			(type default)
+		)
+	)
+	(wire
+		(pts
 			(xy 264.16 85.09) (xy 270.51 85.09)
 		)
@@
 	(wire
 		(pts
+			(xy 201.93 105.41) (xy 190.5 105.41)
+		)
+		(stroke
+			(width 0)
+			(type default)
+		)
+	)
+	(wire
+		(pts
 			(xy 271.78 147.32) (xy 271.78 109.22)
 		)
@@
 	(wire
 		(pts
+			(xy 205.74 93.98) (xy 205.74 97.79)
+		)
+		(stroke
+			(width 0)
+			(type default)
+		)
+	)
+	(wire
+		(pts
 			(xy 228.6 66.04) (xy 231.14 66.04)
 		)
@@
 	(wire
 		(pts
-			(xy 205.74 90.17) (xy 205.74 95.25)
+			(xy 205.74 90.17) (xy 205.74 93.98)
 		)
 		(stroke
@@
 	(wire
 		(pts
+			(xy 190.5 40.64) (xy 190.5 93.98)
+		)
+		(stroke
+			(width 0)
+			(type default)
+		)
+	)
+	(wire
+		(pts
 			(xy 231.14 36.83) (xy 231.14 66.04)
 		)
@@
 	(wire
 		(pts
+			(xy 210.82 93.98) (xy 227.33 93.98)
+		)
+		(stroke
+			(width 0)
+			(type default)
+		)
+	)
+	(wire
+		(pts
 			(xy 270.51 85.09) (xy 270.51 87.63)
 		)
@@
 	(wire
 		(pts
+			(xy 190.5 40.64) (xy 194.31 40.64)
+		)
+		(stroke
+			(width 0)
+			(type default)
+		)
+	)
+	(wire
+		(pts
 			(xy 184.15 142.24) (xy 184.15 82.55)
 		)
@@
 	(wire
 		(pts
-			(xy 205.74 95.25) (xy 218.44 95.25)
+			(xy 227.33 93.98) (xy 227.33 109.22)
 		)
 		(stroke
@@
 					(unit 1)
 				)
+			)
+		)
+	)
+	(symbol
+		(lib_id "Device:L")
+		(at 215.9 101.6 0)
+		(unit 1)
+		(exclude_from_sim no)
+		(in_bom yes)
+		(on_board yes)
+		(dnp no)
+		(fields_autoplaced yes)
+		(property "Reference" "L2"
+			(at 217.17 100.3299 0)
+			(effects
+				(font
+					(size 1.27 1.27)
+				)
+				(justify left)
+			)
+		)
+		(property "Value" "L"
+			(at 217.17 102.8699 0)
+			(effects
+				(font
+					(size 1.27 1.27)
+				)
+				(justify left)
+			)
+		)
+		(property "Footprint" ""
+			(at 215.9 101.6 0)
+			(effects
+				(font
+					(size 1.27 1.27)
+				)
+				(hide yes)
+			)
+		)
+		(property "Datasheet" "~"
+			(at 215.9 101.6 0)
+			(effects
+				(font
+					(size 1.27 1.27)
+				)
+				(hide yes)
+			)
+		)
+		(property "Description" "Inductor"
+			(at 215.9 101.6 0)
+			(effects
+				(font
+					(size 1.27 1.27)
+				)
+				(hide yes)
+			)
+		)
+		(pin "1"
+		)
+		(pin "2"
+		)
+		(instances
+			(project "demo1"
+				(path "/4b72072b-4b2e-4f08-bc1f-9380322b406b"
+					(reference "L2")
+					(unit 1)
+				)
